File: FW2-04-UniversalTimer.brd (EAGLE design)
At the start: 62 x 37 mm, 21 parts, among them IC1 LM555N, Q1 BC557

Commit message: Silkscreen improvements
Parts:
- moved D3 1.27 mm to (39.0, 10.6)
Routing:
- net N$2: track 7.48 -> 25.1 mm
- net N$9: track 0.00 -> 9.42 mm
- net N$12: track 0.00 -> 5.99 mm
- net N$13: track 0.00 -> 3.81 mm
Other:
- board text added: "COM"
- board text added: "NC"
- board text added: "NO"
- board text added: "OUTPUT"
- board text added: "RELAY"
Changed lines of the file:
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@@
 <setting verticaltext="up"/>
 </settings>
-<grid distance="0.05" unitdist="inch" unit="inch" style="lines" multiple="1" display="yes" altdistance="0.005" altunitdist="inch" altunit="inch"/>
+<grid distance="0.01" unitdist="inch" unit="inch" style="lines" multiple="1" display="yes" altdistance="0.005" altunitdist="inch" altunit="inch"/>
 <layers>
 <layer number="1" name="Top" color="4" fill="1" visible="yes" active="yes"/>
@@
 <layer number="23" name="tOrigins" color="15" fill="1" visible="yes" active="yes"/>
 <layer number="24" name="bOrigins" color="15" fill="1" visible="yes" active="yes"/>
-<layer number="25" name="tNames" color="7" fill="1" visible="yes" active="yes"/>
+<layer number="25" name="tNames" color="7" fill="1" visible="no" active="yes"/>
 <layer number="26" name="bNames" color="7" fill="1" visible="no" active="yes"/>
 <layer number="27" name="tValues" color="7" fill="1" visible="no" active="yes"/>
@@
 <text x="59.85" y="9.672" size="1.016" layer="22" font="vector" ratio="16" rot="SMR0">(c) 2016 Freetronics Pty Ltd</text>
 <text x="6.346" y="2.032" size="1.27" layer="21" font="vector" ratio="15" rot="R90">tron.cc/fw2-timer</text>
-<text x="19.828" y="0.656" size="1.8796" layer="21" font="vector" ratio="15">Universal Timer</text>
+<text x="32.782" y="34.798" size="1.778" layer="21" font="vector" ratio="15" align="bottom-center">Universal Timer</text>
 <text x="59.85" y="8.132" size="1.016" layer="22" font="vector" ratio="16" rot="SMR0">Licensed under the TAPR</text>
 <text x="59.85" y="6.862" size="1.016" layer="22" font="vector" ratio="16" rot="SMR0">Open Hardware License</text>
 <text x="59.93" y="5.592" size="1.016" layer="22" font="vector" ratio="16" rot="SMR0">www.tapr.org/OHL</text>
 <text x="59.35" y="1.082" size="1.27" layer="22" font="vector" ratio="16" rot="SMR0">SKU: FW2DOORBELL</text>
-<text x="2.568" y="40.962" size="1.2446" layer="21" font="vector" ratio="15">Compatible with Dick Smith's</text>
-<text x="2.568" y="38.93" size="1.2446" layer="21" font="vector" ratio="15">"Fun Way Into Electronics"</text>
+<text x="20.348" y="2.54" size="1.2446" layer="21" font="vector" ratio="15">Compatible with Dick Smith's</text>
+<text x="20.348" y="0.762" size="1.2446" layer="21" font="vector" ratio="15">"Fun Way Into Electronics"</text>
 <wire x1="18.298" y1="34.34" x2="19.822" y2="34.34" width="0.4064" layer="21"/>
 <wire x1="19.06" y1="35.102" x2="19.06" y2="33.578" width="0.4064" layer="21"/>
@@
 <wire x1="1.565" y1="18.23" x2="1.565" y2="2.99" width="0.4064" layer="21"/>
 <text x="16.4742" y="28.7116" size="1.27" layer="21" font="vector" ratio="15" align="bottom-center">9Vdc</text>
-<text x="34.318" y="38.422" size="1.2446" layer="21" font="vector" ratio="15">Volume 2</text>
-<text x="48.272" y="38.466" size="1.778" layer="21" ratio="13">+</text>
+<text x="48.288" y="0.762" size="1.2446" layer="21" font="vector" ratio="15">Volume 2</text>
+<text x="20.332" y="13.066" size="1.778" layer="21" ratio="13">+</text>
 <wire x1="13.218" y1="34.34" x2="14.742" y2="34.34" width="0.4064" layer="21"/>
 <text x="6.5682" y="28.7116" size="1.27" layer="21" font="vector" ratio="15" align="bottom-center">BUTTON</text>
@@
 <wire x1="1.778" y1="35.052" x2="1.778" y2="28.956" width="0.254" layer="21"/>
 <wire x1="2.54" y1="28.194" x2="1.778" y2="28.956" width="0.254" layer="21" curve="-90"/>
-<text x="51.32" y="37.958" size="1.778" layer="21" ratio="13">+</text>
+<text x="14.49" y="7.478" size="1.778" layer="21" ratio="13">+</text>
 <circle x="32.512" y="4.826" radius="0.359209375" width="0.508" layer="21"/>
 <wire x1="2.18" y1="22.54" x2="2.18" y2="24.54" width="0.254" layer="21"/>
@@
 <wire x1="6.78" y1="22.54" x2="2.18" y2="22.54" width="0.254" layer="21"/>
 <text x="2.01" y="24.85" size="1.27" layer="21">100nF</text>
+<text x="50.8" y="33.7916" size="1.27" layer="21" font="vector" ratio="15" align="bottom-center">COM</text>
+<text x="55.88" y="33.7916" size="1.27" layer="21" font="vector" ratio="15" align="bottom-center">NC</text>
+<text x="45.72" y="33.7916" size="1.27" layer="21" font="vector" ratio="15" align="bottom-center">NO</text>
+<wire x1="57.15" y1="28.194" x2="57.912" y2="28.956" width="0.254" layer="21" curve="90"/>
+<wire x1="44.45" y1="28.194" x2="43.688" y2="28.956" width="0.254" layer="21" curve="-90"/>
+<wire x1="57.912" y1="35.052" x2="57.15" y2="35.814" width="0.254" layer="21" curve="90"/>
+<wire x1="44.45" y1="35.814" x2="43.688" y2="35.052" width="0.254" layer="21" curve="90"/>
+<wire x1="43.688" y1="35.052" x2="43.688" y2="28.956" width="0.254" layer="21"/>
+<wire x1="57.912" y1="35.052" x2="57.912" y2="28.956" width="0.254" layer="21"/>
+<wire x1="44.45" y1="28.194" x2="57.15" y2="28.194" width="0.254" layer="21"/>
+<wire x1="44.45" y1="35.814" x2="57.15" y2="35.814" width="0.254" layer="21"/>
+<text x="47.244" y="28.7116" size="1.27" layer="21" font="vector" ratio="15" align="bottom-center">RELAY</text>
+<text x="54.356" y="28.7116" size="1.27" layer="21" font="vector" ratio="15" align="bottom-center">OUTPUT</text>
 </plain>
 <attributes>
@@
 <element name="JP4" library="freetronics-master-v1.1" package="1X01" value="SPKR-" x="50.8" y="31.75"/>
 <element name="JP3" library="freetronics-master-v1.1" package="1X01" value="SPKR+" x="55.88" y="31.75"/>
-<element name="D3" library="freetronics-2" package="DIODE-1N4001" value="1N4001" x="39.04" y="9.36" rot="R90"/>
+<element name="D3" library="freetronics-2" package="DIODE-1N4001" value="1N4001" x="39.04" y="10.63" rot="R90"/>
 <element name="C1" library="freetronics-2" package="CAP-PTH-SMALL" value="100nF" x="5.78" y="23.54" rot="R180"/>
 <element name="C3" library="freetronics-jon.1" package="CPOL-RADIAL-10UF-25V" value="47uF 6.3V" x="16.51" y="5.08" rot="R90"/>
@@
 <contactref element="R2" pad="P$1"/>
 <contactref element="C2" pad="2"/>
-<wire x1="44.831" y1="9.017" x2="39.04" y2="4.28" width="0.6096" layer="16" curve="-50"/>
-<wire x1="3.81" y1="31.75" x2="13.97" y2="31.75" width="0" layer="19" extent="1-1"/>
-<wire x1="3.24" y1="23.54" x2="3.81" y2="31.75" width="0" layer="19" extent="1-1"/>
+<wire x1="44.831" y1="9.017" x2="39.04" y2="5.55" width="0.6096" layer="16" curve="-50"/>
 <wire x1="17.78" y1="19.05" x2="13.97" y2="31.75" width="0" layer="19" extent="1-1"/>
 <wire x1="15.24" y1="13.97" x2="17.78" y2="19.05" width="0" layer="19" extent="1-1"/>
 <wire x1="16.51" y1="3.81" x2="15.24" y2="13.97" width="0" layer="19" extent="1-1"/>
 <wire x1="10.16" y1="3.81" x2="16.51" y2="3.81" width="0" layer="19" extent="1-1"/>
-<wire x1="39.04" y1="4.28" x2="16.51" y2="3.81" width="0" layer="19" extent="1-1"/>
+<wire x1="39.04" y1="5.55" x2="16.51" y2="3.81" width="0" layer="19" extent="1-1"/>
+<wire x1="3.24" y1="23.54" x2="3.81" y2="31.75" width="0.6096" layer="16" curve="-70"/>
+<wire x1="3.81" y1="31.75" x2="13.97" y2="31.75" width="0.6096" layer="16" curve="-90"/>
 </signal>
 <signal name="N$3">
 <contactref element="RLY1" pad="1"/>
 <contactref element="D3" pad="C"/>
-<wire x1="56.769" y1="9.017" x2="39.04" y2="14.44" width="0.6096" layer="16" curve="30"/>
+<wire x1="56.769" y1="9.017" x2="39.04" y2="15.71" width="0.6096" layer="16" curve="30"/>
 </signal>
 <signal name="N$4">
@@
 <contactref element="Q1" pad="2"/>
 <contactref element="D2" pad="C"/>
-<wire x1="30.48" y1="22.86" x2="35.255" y2="22.05" width="0" layer="19" extent="1-1"/>
-<wire x1="27.94" y1="19.05" x2="30.48" y2="22.86" width="0" layer="19" extent="1-1"/>
+<wire x1="35.255" y1="22.05" x2="30.48" y2="22.86" width="0.6096" layer="16" curve="60"/>
+<wire x1="30.48" y1="22.86" x2="27.94" y2="19.05" width="0.6096" layer="16" curve="70"/>
 </signal>
 <signal name="N$10">
@@
 <contactref element="R3" pad="P$1"/>
 <contactref element="VR1" pad="E"/>
-<wire x1="30.95" y1="26.97" x2="32.87" y2="32.64" width="0" layer="19" extent="1-1"/>
+<wire x1="32.87" y1="32.64" x2="30.95" y2="26.97" width="0.6096" layer="16" curve="50"/>
 </signal>
 <signal name="N$13">
 <contactref element="D2" pad="A"/>
 <contactref element="D1" pad="C"/>
-<wire x1="21.59" y1="22.86" x2="25.4" y2="22.86" width="0" layer="19" extent="1-1"/>
+<wire x1="25.4" y1="22.86" x2="21.59" y2="22.86" width="0.6096" layer="16" curve="20"/>
 </signal>
 </signals>
